Commit message: fixed robot_core_esda.xacro, the thing still sink in ground plane

File: description/robot.urdf.xacro (robot description, xacro)
@@ -3,5 +3,5 @@
     <xacro:arg name="use_ros2_control" default="true"/>
     <xacro:arg name="sim_mode" default="false"/>
-    <xacro:include filename="$(find esda_vehicle_control)/description/robot_core.xacro"/>
+    <xacro:include filename="$(find esda_vehicle_control)/description/robot_core_esda.xacro"/>
     <!--<xacro:include filename="robot_core_esda.xacro" />-->
     <xacro:if value="$(arg use_ros2_control)">
@@ -11,7 +11,7 @@
         <xacro:include filename="$(find esda_vehicle_control)/description/ignition_control.xacro" />
     </xacro:unless>
-    <!--
     <xacro:include filename="lidar.xacro" />
     <xacro:include filename="camera.xacro" />
+    <!--
     <xacro:include filename="depth_camera.xacro" /> -->
     <!--<xacro:include filename="face.xacro" /> -->

File: description/robot_core_esda.xacro (robot description, xacro)
@@ -38,5 +38,5 @@
             <origin xyz="0 0 0" rpy="0 0 0"/>
             <mass value="100"/>
-            <inertia ixx="10" ixy="10" ixz="10" iyy="10" iyz="10" izz="10"/>
+            <inertia ixx="4.507" ixy="0.047271135" ixz="-0.009138455" iyy="1.732" iyz="-0.551074502" izz="5.113"/>
         </inertial>
         <!-- Part fcid_welded_body__configuration_ali_2mm -->

Commit message: fix spawner thing

File: description/robot.urdf.xacro (robot description, xacro)
@@ -13,4 +13,3 @@
     <xacro:include filename="camera.xacro" />
     <!-- <xacro:include filename="depth_camera.xacro" /> -->
-    <xacro:include filename="face.xacro" />
 </robot>

File: description/robot_core_esda.xacro (robot description, xacro)
@@ -14,6 +14,6 @@
     <xacro:property name="caster_wheel_radius" value="0.01"/>
     <xacro:property name="caster_wheel_mass" value="0.45"/>
-    <xacro:property name="caster_wheel_offset_x" value="−0.74898875"/>
-    <xacro:property name="caster_wheel_offset_z" value="−0.082"/>
+    <xacro:property name="caster_wheel_offset_x" value="-0.74898875"/>
+    <xacro:property name="caster_wheel_offset_z" value="-0.082"/>
     <material name="white">
         <color rgba="1 1 1 1" />
@@ -46,5 +46,5 @@
         <parent link="base_link"/>
         <child link="chassis"/>
-        <origin xyz="-0.08353 0 0.0137"/>    <!-- NOTE: the origin is the coordinates of parent link from child link perspective-->
+        <origin xyz="-0.08353 0 0.0137"/>
     </joint>
     <link name="chassis">
@@ -56,5 +56,5 @@
         <!-- Part fcid_welded_body__configuration_ali_2mm -->
         <visual>
-            <origin xyz="-0.4005 0 0.15" rpy="0 0 ${pi/2}"/> <!-- NOTE: origin here is the coordinates of the link from the mesh perspective-->
+            <origin xyz="-0.4005 0 0.15" rpy="0 0 ${pi/2}"/>
             <geometry>
                 <mesh filename="file://$(find esda_vehicle_control)/assets/fcid_welded_body__configuration_ali_2mm.stl"/>
@@ -245,5 +245,5 @@
                 <mesh filename="file://$(find esda_vehicle_control)/assets/drve_arm_bracket.stl"/>
             </geometry>
-        </collision>"
+        </collision>
         	<!-- Part drve_bottom_plate -->
         <visual>
